File: kicad/espclock3.kicad_pcb (KiCad board)
At the start: 2 copper layers, 65.5 x 57.2 mm, 24 parts, among them J1 Quartz Clock, J2 Battery, J5 PCF8563, SW1 SW_Push, U3 ATtiny85-20PU

Commit message: Updated to v3.1
Updated to v3.1
Parts:
- added R8: 47K, Resistor_THT:R_Axial_DIN0309_L9.0mm_D3.2mm_P12.70mm_Horizontal, F.Cu at (80.6, 87.7)
- added R9: 10K, Resistor_THT:R_Axial_DIN0309_L9.0mm_D3.2mm_P12.70mm_Horizontal, F.Cu at (80.6, 83.8)
Connections:
- C1 pad 2: /GND -> Net-(C1-Pad2)
- C2 pad 2: /GND -> Net-(C1-Pad2)
- C4 pad 2: /GND -> Net-(C1-Pad2)
- ESP07-VCC1 pad 7: (no net) -> /ADC
- J2 pad 1: /GND -> Net-(C1-Pad2)
- L1 pad 1: /GND -> Net-(C1-Pad2)
- SW1 pad 1: /GND -> Net-(C1-Pad2)
- U3 pad 4: /GND -> Net-(C1-Pad2)
Routing:
- net Net-(C1-Pad2): track 0.00 -> 88.5 mm
- net Net-(C1-Pad1): track 35.4 -> 83.6 mm
- net /GND: track 123.2 -> 76.6 mm
- net /ADC: track 0.00 -> 32.2 mm
- net /GPIO12: track 53.5 -> 61.3 mm
- net /VCC: track 82.3 -> 85.5 mm
- net /GPIO0: track 54.0 -> 53.1 mm
- net Net-(C4-Pad1): track 79.2 -> 78.4 mm
- net /GPIO16: track 24.7 -> 25.4 mm
